File: boards/v1/iv12-driver-board-v1b.sch (EAGLE design)
At the start: 84 parts, among them J1 85791-4020, J2 SSW-106-02-S-S, J4 SSW-103-02-S-S, J5 SSW-106-02-S-S, Q1 BSS123, U2 HCPL-181-000E, U3 PIC18F67J60-I/PT, U4 25AA02E48T-I/OT

Commit message: changed to correct version of board
Parts:
- removed D4: RED, microbuilder:LED0805_NOOUTLINE
- removed J3: (no value), tag-connect:TC2030-MCP-NL
- removed R16: 27k 1/4w, rcl:R-US_R1206
- added D1: RED, microbuilder:LED0805_NOOUTLINE
- added J6: MOLEX-87758-1016, 0GlenConnectors:CON-2MM-2X5-MOLEX-87758-1016
- added R4: 1k, rcl:R-US_R0805
- R9: value 1k 1/8w -> 51k 1/8w
- renumbered TP_24 to TP_24V
Connections:
- net N$8 renamed VCAP
- removed net BLANK_3V3: J5-2.1
- removed net CLK_3V3: J5-5.1
- removed net DATA_3V3: J5-3.1
- removed net LATCH_3V3: J5-4.1
- removed net N$23: D4.A, R16.2
- removed net NEO_DOUT: U3.RB2/INT2
- removed net VPPIN: R16.1
- new net BLANK: J5-4.1, U3.RB5/KBI1
- new net LATCH: J5-3.1, U3.RC2/ECCP1/P1A
- new net LED3: R27.2, U3.RE5/P1C
- new net N$1: D1.A, R4.1
- net +3V3: now also J5-6.1, J6.3, J6.4; no longer J3.VDD, J5-1.1
- net /MCLR: now also J6.1, J6.2; no longer J3.VPP/MCLR
- net ATFLAG: no longer D4.C
- net GND: now also D1.C, J5-5.1, J6.5, J6.6; no longer J3.VSS(GND), J5-6.1
- net LED1: now also R4.2, U3.RE3/P3C; no longer R26.2, U3.RE4/P3B
- net LED2: now also R26.2, U3.RE4/P3B; no longer R27.2, U3.RE5/P1C
- net MOSI: now also J5-2.1
- net PGC: now also J6.10, J6.9; no longer J3.ICSP_CLK/PGC
- net PGD: now also J6.7, J6.8; no longer J3.ICSP_DAT/PGD
- net SCK: now also J5-1.1
Other:
- note added: "Copyright 2020 by Glen Akins. All rights reserved. This drawing may be shared according to the terms of the GNU General Public License Version 3 or higher."
- note removed: "SPI and WS2812B TO TUBE BOARD"
- moved on the sheet: C15, C33, D10, D11, J5-1, J5-2, J5-3, J5-4, J5-5, J5-6, OSC1, R26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
